Commit message: Using gripper in Gazebo

File: src/desk_cleaner_bringup/urdf/ur5e_desk_cleaner.urdf.xacro (robot description, xacro)
@@ -8,4 +8,5 @@
   <xacro:arg name="safety_limits" default="false"/>
   <xacro:arg name="sim_gazebo" default="false"/>
+  <xacro:arg name="use_fake_hardware" default="true"/>
   <xacro:arg name="initial_positions_file" default="$(find ur_description)/config/initial_positions.yaml"/>
   <xacro:include filename="$(find ur_description)/urdf/ur_macro.xacro"/>
@@ -41,32 +42,32 @@
     <origin xyz="0 0 0" rpy="0 0 0"/>
   </joint>
-  <xacro:if value="${is_humble}">
-    <xacro:ur_robot
-      name="$(arg name)"
-      tf_prefix="$(arg tf_prefix)"
-      parent="desk_pedestal"
-      joint_limits_parameters_file="$(find ur_description)/config/$(arg ur_type)/joint_limits.yaml"
-      kinematics_parameters_file="$(find ur_description)/config/$(arg ur_type)/default_kinematics.yaml"
-      physical_parameters_file="$(find ur_description)/config/$(arg ur_type)/physical_parameters.yaml"
-      visual_parameters_file="$(find ur_description)/config/$(arg ur_type)/visual_parameters.yaml"
-      safety_limits="$(arg safety_limits)"
-      use_fake_hardware="true"
-      fake_sensor_commands="false"
-      sim_gazebo="$(arg sim_gazebo)"
-      generate_ros2_control_tag="true"
-      initial_positions="${xacro.load_yaml(initial_positions_file)}"
-    >
-      <origin xyz="0 0 0.75" rpy="0 0 0"/>
-    </xacro:ur_robot>
-  </xacro:if>
+  <xacro:ur_robot
+    name="$(arg name)"
+    tf_prefix="$(arg tf_prefix)"
+    parent="desk_pedestal"
+    joint_limits_parameters_file="$(find ur_description)/config/$(arg ur_type)/joint_limits.yaml"
+    kinematics_parameters_file="$(find ur_description)/config/$(arg ur_type)/default_kinematics.yaml"
+    physical_parameters_file="$(find ur_description)/config/$(arg ur_type)/physical_parameters.yaml"
+    visual_parameters_file="$(find ur_description)/config/$(arg ur_type)/visual_parameters.yaml"
+    safety_limits="$(arg safety_limits)"
+    use_fake_hardware="$(arg use_fake_hardware)"
+    fake_sensor_commands="false"
+    sim_gazebo="$(arg sim_gazebo)"
+    generate_ros2_control_tag="true"
+    initial_positions="${xacro.load_yaml(initial_positions_file)}"
+  >
+    <origin xyz="0 0 0.75" rpy="0 0 0"/>
+  </xacro:ur_robot>
   <xacro:ur_to_robotiq
     prefix="$(arg tf_prefix)"
-    connected_to="$(arg tf_prefix)tool0"
+    parent="$(arg tf_prefix)tool0"
+    child="$(arg tf_prefix)gripper_mount_link"
   />
   <xacro:robotiq_gripper
-    name="RobotiqGripperHardwareInterface"
+    name="RobotiqGripperHardware"
     prefix="$(arg tf_prefix)"
     parent="$(arg tf_prefix)gripper_mount_link"
-    use_fake_hardware="true"
+    use_fake_hardware="$(arg use_fake_hardware)"
+    sim_gazebo="$(arg sim_gazebo)"
     include_ros2_control="true"
     com_port="/dev/ttyUSB0"
