Commit message: Update urdf to include gazebo ros2 control plugin. Also update urdf for gazebo to display meshes (not too sure what is wrong with the original implementations). Update srdf for some collision scenario. Include a launch file similar to ur5e_gazebo.launch.py for robot so101

File: src/desk_cleaner_description/so101/urdf/ros2_control/so101_ros2_control.xacro (robot description, xacro)
@@ -26,4 +26,5 @@
         variant:='follower'
         hardware_type:='mock'
+        sim_gazebo:='false'
         usb_port:='/dev/ttyUSB0'
         joint_config_file:=''
@@ -31,12 +32,17 @@
         <ros2_control name="${system_name}" type="system">
               <hardware>
-                <xacro:if value="${hardware_type == 'mock'}">
-                    <plugin>mock_components/GenericSystem</plugin>
+                <xacro:if value="${sim_gazebo}">
+                    <plugin>gazebo_ros2_control/GazeboSystem</plugin>
                 </xacro:if>
-                <xacro:if value="${hardware_type == 'real'}">
-                    <plugin>feetech_ros2_driver/FeetechHardwareInterface</plugin>
-                    <param name="usb_port">${usb_port}</param>
-                    <param name="joint_config_file">${joint_config_file}</param>
-                </xacro:if>
+                <xacro:unless value="${sim_gazebo}">
+                    <xacro:if value="${hardware_type == 'mock'}">
+                        <plugin>mock_components/GenericSystem</plugin>
+                    </xacro:if>
+                    <xacro:if value="${hardware_type == 'real'}">
+                        <plugin>feetech_ros2_driver/FeetechHardwareInterface</plugin>
+                        <param name="usb_port">${usb_port}</param>
+                        <param name="joint_config_file">${joint_config_file}</param>
+                    </xacro:if>
+                </xacro:unless>
             </hardware>
             <!-- arm joints -->

File: src/desk_cleaner_description/so101/urdf/so101_arm.urdf.xacro (robot description, xacro)
@@ -2,8 +2,9 @@
 <robot name="so101_arm" xmlns:xacro="http://www.ros.org/wiki/xacro">
   <xacro:arg name="variant" default="follower"/>          <!-- leader | follower -->
-  <xacro:arg name="mesh_dir" default="package://desk_cleaner_description/so101/meshes"/>
+  <xacro:arg name="mesh_dir" default="file://$(find desk_cleaner_description)/so101/meshes"/>
   <xacro:arg name="add_transmissions" default="false"/>
   <xacro:arg name="use_ros2_control" default="true"/>
   <xacro:arg name="hardware_type" default="mock"/>
+  <xacro:arg name="sim_gazebo" default="false"/>
   <xacro:arg name="usb_port" default="/dev/ttyUSB0"/>
   <xacro:arg name="joint_config_file" default=""/>
@@ -20,4 +21,5 @@
   <xacro:property name="enable_static_cam" value="$(arg enable_static_cam)"/>
   <xacro:property name="enable_wrist_cam" value="$(arg enable_wrist_cam)"/>
+  <xacro:property name="sim_gazebo" value="$(arg sim_gazebo)"/>
   <xacro:include filename="$(find desk_cleaner_description)/so101/urdf/so101_macros.xacro"/>
   <xacro:include filename="$(find desk_cleaner_description)/so101/urdf/so101_materials.xacro"/>
@@ -29,7 +31,13 @@
   <!-- <xacro:include filename="$(find desk_cleaner_description)/so101/urdf/so101_cameras.xacro"/> -->
   <xacro:so101_materials/>
+  <link name="world"/>
   <xacro:so101_arm_common
     mesh_dir="$(arg mesh_dir)"
     add_transmissions="$(arg add_transmissions)"/>
+  <joint name="world_to_base_link" type="fixed">
+    <parent link="world"/>
+    <child link="base_link"/>
+    <origin xyz="0 0 0" rpy="0 0 0"/>
+  </joint>
   <xacro:if value="${variant == 'leader'}">
     <xacro:so101_ee_leader
@@ -46,4 +54,5 @@
       variant="${variant}"
       hardware_type="$(arg hardware_type)"
+      sim_gazebo="$(arg sim_gazebo)"
       usb_port="$(arg usb_port)"
       joint_config_file="$(arg joint_config_file)"
@@ -61,3 +70,10 @@
       rpy="$(arg cam_wrist_rpy)"/>
   </xacro:if> -->
+  <xacro:if value="$(arg sim_gazebo)">
+    <gazebo>
+      <plugin filename="libgazebo_ros2_control.so" name="gazebo_ros2_control">
+        <parameters>$(find desk_cleaner_bringup)/config/so101_controllers.yaml</parameters>
+      </plugin>
+    </gazebo>
+  </xacro:if>
 </robot>
